File: SLKCAN/KiCad/SLKCAN.kicad_pcb (KiCad board)
At the start: 4 copper layers, 95.3 x 47 mm, 46 parts, among them J1 FTDI, J2 POWER & CAN, J3 TF-15X15, J4 AUX, SW1 SW_Push, U1 AMS1117-3.3, U2 LD1085V50, U3 ESP32-WROOM-32, U4 MCP2515-xSO, U5 MCP2551-I-SN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

Commit message: Fixes from SLKCAN01 known issues
Fixes from SLKCAN01 known issues.
Parts:
- U6: value LSF0204PWR -> TXS0104EPWR
- turned R6 to 270 degrees
Connections:
- D2 pad 1: +3V3 -> Net-(D2-Pad1)
- D2 pad 2: Net-(D2-Pad2) -> +3V3
- J4 pad 9: AUX8 -> CAN_*INT
- R6 pad 1: Net-(D2-Pad2) -> Net-(D2-Pad1)
- U3 pad 26: CAN_*INT -> Net-(U3-Pad26)
- U3 pad 7: AUX8 -> CAN_*INT
Routing:
- net AUX8: track 37.2 -> 0.00 mm, vias 2 -> 0
- net CAN_*INT: track 37.4 -> 69.0 mm, vias 2 -> 5
- net Net-(D2-Pad1): track 0.00 -> 4.77 mm, vias 0 -> 1
- net Net-(D2-Pad2): track 2.55 -> 0.00 mm
- net Net-(R6-Pad2): track 11.1 -> 9.78 mm
Other:
- board text added: "INT"
- board text added: "SLKCAN02"
- board text removed: "35"
- board text removed: "SLKCAN01"
