File: SLKCAN/KiCad/SLKCAN.sch (KiCad schematic (older format))
At the start: 46 parts, among them J1 FTDI, J2 POWER & CAN, J3 TF-15X15, J4 AUX, SW1 SW_Push, U1 AMS1117-3.3, U2 LD1085V50, U3 ESP32-WROOM-32, U4 MCP2515-xSO, U5 MCP2551-I-SN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

Commit message: Fixes from SLKCAN01 known issues
Fixes from SLKCAN01 known issues.
Parts:
- J3: symbol TF-15X15:TF-15X15 -> SLKCAN-rescue:TF-15X15-TF-15X15
- U2: symbol ld1085v50:LD1085V50 -> SLKCAN-rescue:LD1085V50-ld1085v50
- U6: value LSF0204PWR -> TXS0104EPWR; symbol LSF0204PWR:LSF0204PWR -> SLKCAN-rescue:LSF0204PWR-LSF0204PWR
Connections:
- net AUX8 is gone; now on net CAN_*INT: J4.9 (Pin_9), U3.7 (IO35)
- net +3V3: now also D2.2 (A); no longer D2.1 (K)
- net CAN_*INT: no longer U3.26 (IO4)
- net at R6.1: now also D2.1 (K); no longer D2.2 (A)
Other:
- note added: "SLKCAN01\n20210303/CZM - Moved CAN SPI to HSPI\n20210303/CZM - Added LSF Level Translator for CAN SPI\n20210303/CZM - Moved 3.3V reg downstream of 5v reg.\n20210303/CZM - Added optional MicroSD card slot. VPSI.\n20210303/CZM - Added option CAN termination.\n20210303/CZM - Added Decoupling caps to MCP chips.\n20210303/CZM - Moved FTDI pin 3 from 3.3v to 5V. jumper.\n20210303/CZM - Added heartbeat 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"
- note removed: "20210303/CZM - Moved CAN SPI to HSPI\n20210303/CZM - Added LSF Level Translator for CAN SPI\n20210303/CZM - Moved 3.3V reg downstream of 5v reg.\n20210303/CZM - Added optional MicroSD card slot. VPSI.\n20210303/CZM - Added option CAN termination.\n20210303/CZM - Added Decoupling caps to MCP chips.\n20210303/CZM - Moved FTDI pin 3 from 3.3v to 5V. jumper.\n20210303/CZM - Added heartbeat LED.\n2021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"
- moved on the sheet: D2
Changed lines of the file:
@@
 Sheet 1 1
 Title "SLKCAN"
-Date "2021-03-13"
-Rev "01"
+Date "2021-06-15"
+Rev "02"
 Comp "Auther: CZ Morris"
 Comment1 "Experimental CANBUS Interface, ESP32"
 Comment2 ""
 Comment3 ""
-Comment4 "RELEASE DRAFT 20210313"
+Comment4 "PRE-RELEASE"
 $EndDescr
 $Comp
@@
 Text GLabel 10000 2350 2    50   Input ~ 0
 UART0_RXD
-Text GLabel 10000 2450 2    50   Input ~ 0
+Text GLabel 4150 3950 0    50   Input ~ 0
 CAN_*INT
 Wire Wire Line
@@
 Wire Wire Line
 	9750 2350 10000 2350
-Wire Wire Line
-	9750 2450 10000 2450
 $Comp
 L Device:R R1
@@
 	9150 4700 9150 4650
 $Comp
-L LSF0204PWR:LSF0204PWR U6
+L SLKCAN-rescue:LSF0204PWR-LSF0204PWR U6
 U 1 1 606673F7
 P 2900 7850
 F 0 "U6" H 2900 8700 50  0000 C CNN
-F 1 "LSF0204PWR" H 2900 8600 50  0000 C CNN
+F 1 "TXS0104EPWR" H 2900 8600 50  0000 C CNN
 F 2 "SOP65P640X120-14N" H 2900 7850 50  0001 L BNN
 F 3 "" H 2900 7850 50  0001 L BNN
@@
 	1500 6750 1500 7350
 $Comp
-L TF-15X15:TF-15X15 J3
+L SLKCAN-rescue:TF-15X15-TF-15X15 J3
 U 1 1 60CB97F8
 P 13800 2000
@@
 F 3 "~" H 11050 2450 50  0001 C CNN
 	1    11050 2450
-	0    1    1    0
-$EndComp
-Wire Wire Line
-	11050 2250 11050 2300
+	0    -1   -1   0
+$EndComp
 Wire Wire Line
 	11050 2600 11050 2650
@@
 CANBUS INTERFACE
 Text Notes 12700 9200 0    59   ~ 0
-20210303/CZM - Moved CAN SPI to HSPI\n20210303/CZM - Added LSF Level Translator for CAN SPI\n20210303/CZM - Moved 3.3V reg downstream of 5v reg.\n20210303/CZM - Added optional MicroSD card slot. VPSI.\n20210303/CZM - Added option CAN termination.\n20210303/CZM - Added Decoupling caps to MCP chips.\n20210303/CZM - Moved FTDI pin 3 from 3.3v to 5V. jumper.\n20210303/CZM - Added heartbeat LED.\n20210303/CZM - Added MCP2551 Rs pull down.\n20210307/CZM - Added extra pins and power to AUX connector\n20210307/CZM - Missing note: Fixed RX pin from FTDI to ESP32\n20210313/CZM - Replaced the AMS 5v reg with a more beefy regulator. \n20210313/CZM - 15uF power inductors on all input lines. SLK bus is very noisy
+SLKCAN01\n20210303/CZM - Moved CAN SPI to HSPI\n20210303/CZM - Added LSF Level Translator for CAN SPI\n20210303/CZM - Moved 3.3V reg downstream of 5v reg.\n20210303/CZM - Added optional MicroSD card slot. VPSI.\n20210303/CZM - Added option CAN termination.\n20210303/CZM - Added Decoupling caps to MCP chips.\n20210303/CZM - Moved FTDI pin 3 from 3.3v to 5V. jumper.\n20210303/CZM - Added heartbeat LED.\n20210303/CZM - Added MCP2551 Rs pull down.\n20210307/CZM - Added extra pins and power to AUX connector\n20210307/CZM - Missing note: Fixed RX pin from FTDI to ESP32\n20210313/CZM - Replaced the AMS 5v reg with a more beefy regulator. \n20210313/CZM - 15uF power inductors on all input lines. SLK bus is very noisy\nSLKCAN02\n20210615/CZM - Disconnected IO4 from CAN_*INT\n20210615/CZM - AUX8 replaced with CAN_*INT\n20210615/CZM - U6 changed to TXS0104EPWR\n
 Text Notes 11150 7150 0    39   ~ 0
 Optional CAN\nTermination
@@
 Wire Wire Line
 	10000 4250 9750 4250
-Text GLabel 10000 4350 2    39   Input ~ 0
-AUX8
-Wire Wire Line
-	9750 4350 10000 4350
 $Comp
 L Connector_Generic:Conn_02x06_Odd_Even J4
@@
 Wire Wire Line
 	4750 3850 5000 3850
-Text GLabel 4050 3950 0    39   Input ~ 0
-AUX8
-Wire Wire Line
-	4050 3950 4250 3950
 $Comp
 L power:+3.3V #PWR0101
@@
 Unused GPIO
 $Comp
-L ld1085v50:LD1085V50 U2
+L SLKCAN-rescue:LD1085V50-ld1085v50 U2
 U 1 1 60513054
 P 4250 1850
@@
 Wire Wire Line
 	2700 2250 3050 2250
+Wire Wire Line
+	4150 3950 4250 3950
+Text GLabel 10000 4350 2    50   Input ~ 0
+CAN_*INT
+Wire Wire Line
+	10000 4350 9750 4350
+Wire Wire Line
+	11050 2250 11050 2300
 $EndSCHEMATC
